File: Hardware/Left/santo_left.sch (KiCad schematic (older format))
At the start: 63 parts, among them J1 USB_C_Receptacle, J2 USB_C_Receptacle, SW1 SW_Push, U1 ATMEGA32U4-MU

Commit message: lable and cleanup
Parts:
- gave numbers to parts that had none: 48
Connections:
- net Row_2: now reaches SW12.1, SW16.1, SW20.1, SW24.1, SW4.1, SW8.1, U1.10 ((PDI/MOSI/PCINT2)PB2)
- net Row_3: now reaches SW13.1, SW17.1, SW21.1, SW25.1, SW5.1, SW9.1, U1.11 ((PDO/MISO/PCINT3)PB3)
- net Column_3: now reaches D14.1 (K), D15.1 (K), D16.1 (K), D17.1 (K), U1.12 ((OC0A/OC1C/~RTS~/PCINT7)PB7)
- net Column_0: now reaches D2.1 (K), D3.1 (K), D4.1 (K), D5.1 (K), U1.28 ((ADC11/PCINT4)PB4)
- net Column_1: now reaches D6.1 (K), D7.1 (K), D8.1 (K), D9.1 (K), U1.29 ((ADC12/OC1A/~OC4B~/PCINT12)PB5)
- net Column_2: now reaches D10.1 (K), D11.1 (K), D12.1 (K), D13.1 (K), U1.30 ((ADC13/OC1B/OC4B/PCINT13)PB6)
- net Column_4: now reaches D18.1 (K), D19.1 (K), D20.1 (K), D21.1 (K), U1.31 ((OC3A/~OC4A~)PC6)
- net Column_5: now reaches D22.1 (K), D23.1 (K), D24.1 (K), D25.1 (K), U1.32 ((ICP3/CLK0/OC4A)PC7)
- net Row_0: now reaches SW10.1, SW14.1, SW18.1, SW2.1, SW22.1, SW6.1, U1.8 ((SS/PCINT0)PB0)
- net Row_1: now reaches SW11.1, SW15.1, SW19.1, SW23.1, SW3.1, SW7.1, U1.9 ((SCLK/PCINT1)PB1)
- no-connect marks 0 -> 27
